File: electronics/kicad/TundraStylus_PCB_Rev01.kicad_pcb (KiCad board)
At the start: 2 copper layers, 80 x 16 mm, 11 parts, among them J1 CON_TPAD, J2 CON_MENU, J3 CON_TRIG, J4 CON_GRIP, SW1 TPAD, SW2 MENU, SW3 TRIG, SW4 GRIP

Commit message: Update pcb files
Other:
- board text added: "GRIP"
- board text added: "MENU"
- board text added: "TPAD"
- board text added: "TRIG"
- board text added: "TUNDRA STYLUS PCB REV01"
Changed lines of the file:
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@@
     (pad_to_mask_clearance 0)
     (pcbplotparams
-      (layerselection 0x0000000_7fffffff)
+      (layerselection 0x00010a0_7fffffff)
       (plot_on_all_layers_selection 0x0001000_00000000)
       (disableapertmacros false)
@@
       (psnegative false)
       (psa4output false)
-      (plotreference false)
+      (plotreference true)
       (plotvalue false)
       (plotinvisibletext false)
@@
       (drillshape 0)
       (scaleselection 1)
-      (outputdirectory "Gerbers/")
+      (outputdirectory "../../gerbers/jlcpcb/")
     )
   )
@@
     (property "ki_keywords" "switch normally-open pushbutton push-button button tactile spst single pole single throw B3SN-3112P")
     (attr smd)
-    (fp_text reference "SW3" (at 0 -4 90) (layer "F.SilkS")
+    (fp_text reference "SW3" (at 0 3.9 90) (layer "F.SilkS")
         (effects (font (size 1 1) (thickness 0.15)))
     )
@@
     (property "ki_keywords" "single row male connector")
     (attr smd)
-    (fp_text reference "J1" (at -2.1 -0.1) (layer "F.SilkS")
+    (fp_text reference "J1" (at -2.1 0.5) (layer "F.SilkS")
         (effects (font (size 1 1) (thickness 0.15)) (justify left))
     )
@@
     (property "ki_keywords" "single row male connector")
     (attr smd)
-    (fp_text reference "J2" (at 3.8 -0.1) (layer "F.SilkS")
+    (fp_text reference "J2" (at 3.8 -0.5) (layer "F.SilkS")
         (effects (font (size 1 1) (thickness 0.15)) (justify right))
     )
@@
     (property "ki_keywords" "single row male connector")
     (attr smd)
-    (fp_text reference "J3" (at 3.7 2.8) (layer "F.SilkS")
+    (fp_text reference "J3" (at 3.7 2) (layer "F.SilkS")
         (effects (font (size 1 1) (thickness 0.15)) (justify right))
     )
@@
     (property "ki_keywords" "single row male connector")
     (attr smd)
-    (fp_text reference "J4" (at -2 2.5) (layer "F.SilkS")
+    (fp_text reference "J4" (at -2 2.9) (layer "F.SilkS")
         (effects (font (size 1 1) (thickness 0.15)) (justify left))
     )
@@
     (property "ki_keywords" "switch normally-open pushbutton push-button button tactile spst single pole single throw B3SN-3112P")
     (attr smd)
-    (fp_text reference "SW4" (at 0 -4 90) (layer "F.SilkS")
+    (fp_text reference "SW4" (at 0 3.9 -90) (layer "F.SilkS")
         (effects (font (size 1 1) (thickness 0.15)))
     )
@@
   (gr_line (start 175 98) (end 95 98)
     (stroke (width 0.1) (type default)) (layer "User.3"))
+  (gr_text "MENU\n" (at 169.6 94) (layer "F.SilkS")
+    (effects (font (size 0.8 0.8) (thickness 0.1)) (justify left bottom))
+  )
+  (gr_text "TUNDRA\nSTYLUS\nPCB\nREV01" (at 125 98.2) (layer "F.SilkS")
+    (effects (font (size 1 1) (thickness 0.15)))
+  )
+  (gr_text "GRIP\n" (at 157 94.2) (layer "F.SilkS")
+    (effects (font (size 0.8 0.8) (thickness 0.1)) (justify left bottom))
+  )
+  (gr_text "TPAD" (at 166.8 104.4) (layer "F.SilkS")
+    (effects (font (size 0.8 0.8) (thickness 0.1)) (justify left bottom))
+  )
+  (gr_text "TRIG" (at 153.4 104.4) (layer "F.SilkS")
+    (effects (font (size 0.8 0.8) (thickness 0.1)) (justify left bottom))
+  )
   (dimension (type aligned) (layer "User.1")
     (pts (xy 99 98) (xy 95 98))

Commit message: Add latest electronics design
Parts:
- removed J3: CON_TRIG, fab:PinHeader_1x02_P2.54mm_Horizontal_SMD
- removed J4: CON_GRIP, fab:PinHeader_1x02_P2.54mm_Horizontal_SMD
- added H4: ~, fab:MountingHole_M2, F.Cu at (92.0, 108.0)
- added H5: ~, fab:MountingHole_M2, F.Cu at (178.0, 88.0)
- added H6: ~, fab:MountingHole_M2, F.Cu at (178.0, 108.0)
- added P1: IO, TundraIO:Conn_FFC_1x05_P1mm_SideEntry_GCT_FFC3B11-05-T, B.Cu at (168.7, 98.0)
- H2: footprint fab:MountingHole_M2.5 -> fab:MountingHole_M2
- J1: value CON_TPAD -> HAPT; footprint fab:PinHeader_1x02_P2.54mm_Horizontal_SMD -> TundraIO:Conn_2pos_Plain; moved to B.Cu
- J2: value CON_MENU -> HAPT; footprint fab:PinHeader_1x02_P2.54mm_Horizontal_SMD -> TundraIO:Conn_2pos_Plain
- moved H2 79.6 mm to (92.0, 88.0), turned to 0 degrees
- moved J2 69.6 mm to (98.0, 94.0), turned to 90 degrees
- moved J1 10.3 mm to (160.0, 93.9), turned to 90 degrees
- moved H1 6.00 mm to (155.0, 98.0)
Connections:
- J1 pad 1: TPAD_A -> HAPT_P
- J1 pad 2: TPAD_B -> HAPT_N
- J2 pad 1: MENU_A -> HAPT_P
- J2 pad 2: MENU_B -> HAPT_N
- SW1 pad 1: TPAD_A -> TPAD
- SW1 pad 2: TPAD_B -> PWR_GND
- SW2 pad 1: MENU_A -> MENU
- SW2 pad 2: MENU_B -> PWR_GND
- SW3 pad 1: TRIG_A -> TRIG
- SW3 pad 2: TRIG_B -> PWR_GND
- SW4 pad 1: GRIP_A -> GRIP
- SW4 pad 2: GRIP_B -> PWR_GND
Routing:
- net HAPT_P: track 0.00 -> 62.8 mm, vias 0 -> 1
- net HAPT_N: track 0.00 -> 62.3 mm, vias 0 -> 1
- net TRIG: track 0.00 -> 61.1 mm, vias 0 -> 1
- net GRIP: track 0.00 -> 50.7 mm, vias 0 -> 1
- net TRIG_B: track 48.0 -> 0.00 mm
- net TRIG_A: track 44.3 -> 0.00 mm
- net GRIP_B: track 41.1 -> 0.00 mm
- net TPAD_B: track 37.5 -> 0.00 mm
- net GRIP_A: track 37.4 -> 0.00 mm
- net TPAD: track 0.00 -> 35.3 mm, vias 0 -> 1
- net TPAD_A: track 33.6 -> 0.00 mm
- net MENU_B: track 29.6 -> 0.00 mm
- net MENU_A: track 25.7 -> 0.00 mm
- net MENU: track 0.00 -> 24.2 mm, vias 0 -> 1
- net PWR_GND: track 0.00 -> 3.88 mm, vias 0 -> 1
- added copper zone on F.Cu, net PWR_GND
Other:
- board size 80 x 16 mm -> 80 x 14 mm
- board text added: "TUNDRA STYLUS PCB REV02"
- board text removed: "GRIP"
- board text removed: "MENU"
- board text removed: "TPAD"
- board text removed: "TRIG"
- board text removed: "TUNDRA STYLUS PCB REV01"
